File: KiCAD/circuit/thermistor.sch (KiCad schematic (older format))
At the start: 24 parts, among them J1 To USB-UART converter, J10 Jumper, J11 Jumper, J12 Jumper, J13 Jumper, J14 Jumper, J15 Jumper, J16 Jumper, J2 Pin header, J3 Pin header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

Commit message: circuit update
Parts:
- added J? (x4): Jumper, symbol Conn_01x01_Female
- added R?: 10k, symbol R
- added U?: FSR, symbol FSR
Connections:
- new net 4: J?.1 (Pin_1), J?.1 (Pin_1), R?.1, R?.2
- new net 4a: J?.1 (Pin_1), U?.1
- new net 4b: J?.1 (Pin_1), U?.2
Other:
- moved on the sheet: J1, J10, J11, J12, J13, J14, J15, J16, J2, J3, J4, J5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

Commit message: update
Parts:
- added C1: 0.1u, symbol C_Small
- gave numbers to parts that had none: 6
Connections:
- net +5V: now also C1.2
- net at J4.1b (Pin_1b), J4.2b (Pin_2b), J4.3b (Pin_3b)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: now also C1.1
Other:
- moved on the sheet: R1
Changed lines of the file:
@@
 L R R1
 U 1 1 5AC420FC
-P 4250 3000
-F 0 "R1" V 4330 3000 50  0000 C CNN
-F 1 "51k" V 4250 3000 50  0000 C CNN
-F 2 "" V 4180 3000 50  0001 C CNN
-F 3 "" H 4250 3000 50  0001 C CNN
-	1    4250 3000
+P 4150 3000
+F 0 "R1" V 4230 3000 50  0000 C CNN
+F 1 "51k" V 4150 3000 50  0000 C CNN
+F 2 "" V 4080 3000 50  0001 C CNN
+F 3 "" H 4150 3000 50  0001 C CNN
+	1    4150 3000
 	0    1    1    0
 $EndComp
@@
 $EndComp
 Wire Wire Line
-	3150 1850 4500 1850
-Wire Wire Line
-	4500 1850 7500 1850
+	3150 1850 4400 1850
+Wire Wire Line
+	4400 1850 7500 1850
 Wire Wire Line
 	7500 1850 7600 1850
@@
 	9550 4750 9550 4700
 Wire Wire Line
-	4500 1850 4500 3000
-Wire Wire Line
-	4400 3000 4500 3000
-Wire Wire Line
-	4500 3000 4650 3000
-Connection ~ 4500 3000
-Wire Wire Line
-	4100 3000 4000 3000
-Wire Wire Line
-	4000 3000 4000 3300
-Wire Wire Line
-	4000 3300 4650 3300
+	4400 1850 4400 3000
+Wire Wire Line
+	4300 3000 4400 3000
+Wire Wire Line
+	4400 3000 4550 3000
+Wire Wire Line
+	4550 3000 4650 3000
+Connection ~ 4400 3000
+Wire Wire Line
+	3850 3000 4000 3000
+Wire Wire Line
+	3850 3000 3850 3300
+Wire Wire Line
+	3850 3300 4650 3300
 Wire Wire Line
 	6600 3300 7800 3300
@@
 Connection ~ 7700 4450
 Wire Wire Line
-	6600 3000 7100 3000
+	6600 3000 6700 3000
+Wire Wire Line
+	6700 3000 7100 3000
 Connection ~ 7100 4450
 Wire Wire Line
@@
 Wire Wire Line
 	3150 2850 3150 4350
-Connection ~ 4500 1850
+Connection ~ 4400 1850
 Wire Wire Line
 	3050 3850 3650 3850
@@
 Connection ~ 3650 4200
 $Comp
-L FSR U?
+L FSR U2
 U 1 1 5AC69E47
 P 9650 6000
-F 0 "U?" H 9500 6400 60  0000 C CNN
+F 0 "U2" H 9500 6400 60  0000 C CNN
 F 1 "FSR" H 9500 6300 60  0000 C CNN
 F 2 "" H 9700 6000 60  0001 C CNN
@@
 $EndComp
 $Comp
-L Conn_01x01_Female J?
+L Conn_01x01_Female J19
 U 1 1 5AC69ED3
 P 8350 5850
-F 0 "J?" H 8350 5950 50  0000 C CNN
+F 0 "J19" H 8350 5950 50  0000 C CNN
 F 1 "Jumper" H 8350 5750 50  0000 C CNN
 F 2 "" H 8350 5850 50  0001 C CNN
@@
 $EndComp
 $Comp
-L Conn_01x01_Female J?
+L Conn_01x01_Female J20
 U 1 1 5AC69F5F
 P 8350 6150
-F 0 "J?" H 8350 6250 50  0000 C CNN
+F 0 "J20" H 8350 6250 50  0000 C CNN
 F 1 "Jumper" H 8350 6050 50  0000 C CNN
 F 2 "" H 8350 6150 50  0001 C CNN
@@
 4b
 $Comp
-L R R?
+L R R6
 U 1 1 5AC6B1CA
 P 9000 2900
-F 0 "R?" V 9080 2900 50  0000 C CNN
+F 0 "R6" V 9080 2900 50  0000 C CNN
 F 1 "10k" V 9000 2900 50  0000 C CNN
 F 2 "" V 8930 2900 50  0001 C CNN
@@
 $EndComp
 $Comp
-L Conn_01x01_Female J?
+L Conn_01x01_Female J17
 U 1 1 5AC6B1D0
 P 8350 2750
-F 0 "J?" H 8350 2850 50  0000 C CNN
+F 0 "J17" H 8350 2850 50  0000 C CNN
 F 1 "Jumper" H 8350 2650 50  0000 C CNN
 F 2 "" H 8350 2750 50  0001 C CNN
@@
 $EndComp
 $Comp
-L Conn_01x01_Female J?
+L Conn_01x01_Female J18
 U 1 1 5AC6B1D6
 P 8350 3050
-F 0 "J?" H 8350 3150 50  0000 C CNN
+F 0 "J18" H 8350 3150 50  0000 C CNN
 F 1 "Jumper" H 8350 2950 50  0000 C CNN
 F 2 "" H 8350 3050 50  0001 C CNN
@@
 Text Label 8800 3050 0    60   ~ 0
 4
+$Comp
+L C_Small C1
+U 1 1 5AC759C2
+P 5650 2600
+F 0 "C1" H 5660 2670 50  0000 L CNN
+F 1 "0.1u" H 5660 2520 50  0000 L CNN
+F 2 "" H 5650 2600 50  0001 C CNN
+F 3 "" H 5650 2600 50  0001 C CNN
+	1    5650 2600
+	0    1    1    0
+$EndComp
+Wire Wire Line
+	5750 2600 6700 2600
+Wire Wire Line
+	6700 2600 6700 3000
+Connection ~ 6700 3000
+Wire Wire Line
+	4550 3000 4550 2600
+Wire Wire Line
+	4550 2600 5550 2600
+Connection ~ 4550 3000
 $EndSCHEMATC
