File: KiCAD/circuit/open_drain.sch (KiCad schematic (older format))
At the start: 13 parts, among them J1 To 9V battery, J2 To Raspberry Pi's GPIO, Q1 2SK2232

Commit message: update
Parts:
- R1, R2, R3, R4, R5, R6: value R -> 470
Changed lines of the file:
@@
 P 7750 3050
 F 0 "R1" V 7830 3050 50  0000 C CNN
-F 1 "R" V 7750 3050 50  0000 C CNN
+F 1 "470" V 7750 3050 50  0000 C CNN
 F 2 "" V 7680 3050 50  0001 C CNN
 F 3 "" H 7750 3050 50  0001 C CNN
@@
 P 7750 3250
 F 0 "R2" V 7830 3250 50  0000 C CNN
-F 1 "R" V 7750 3250 50  0000 C CNN
+F 1 "470" V 7750 3250 50  0000 C CNN
 F 2 "" V 7680 3250 50  0001 C CNN
 F 3 "" H 7750 3250 50  0001 C CNN
@@
 P 7750 3450
 F 0 "R3" V 7830 3450 50  0000 C CNN
-F 1 "R" V 7750 3450 50  0000 C CNN
+F 1 "470" V 7750 3450 50  0000 C CNN
 F 2 "" V 7680 3450 50  0001 C CNN
 F 3 "" H 7750 3450 50  0001 C CNN
@@
 P 7750 3750
 F 0 "R4" V 7830 3750 50  0000 C CNN
-F 1 "R" V 7750 3750 50  0000 C CNN
+F 1 "470" V 7750 3750 50  0000 C CNN
 F 2 "" V 7680 3750 50  0001 C CNN
 F 3 "" H 7750 3750 50  0001 C CNN
@@
 P 7750 3950
 F 0 "R5" V 7830 3950 50  0000 C CNN
-F 1 "R" V 7750 3950 50  0000 C CNN
+F 1 "470" V 7750 3950 50  0000 C CNN
 F 2 "" V 7680 3950 50  0001 C CNN
 F 3 "" H 7750 3950 50  0001 C CNN
@@
 P 7750 4150
 F 0 "R6" V 7830 4150 50  0000 C CNN
-F 1 "R" V 7750 4150 50  0000 C CNN
+F 1 "470" V 7750 4150 50  0000 C CNN
 F 2 "" V 7680 4150 50  0001 C CNN
 F 3 "" H 7750 4150 50  0001 C CNN
